File: hardware/gio/gio.kicad_sch (KiCad schematic)
At the start: 55 parts, among them J1 PJ3001F, J2 PJ3001F, J3 oled, J4 eurorack power, J5 PJ3001F, J6 PJ3001F, SW1 encoder, U1 TL072, U2 MCP3208, U3 DAC8552, U4 XIAO-RP2350-DIP, U5 TL072, U6 AMS1117CD-5.0, U7 REF3040

Commit message: KiCad layout: PCB project moved to hardware/gio/, .gitignore for fab cruft
Project renamed and relocated from hardware/gio-opamp/ to hardware/gio/
to reflect that this is the gio module's main board (the "opamp" suffix
was a holdover from when the project covered just the input op-amp
section). Active files now under hardware/gio/:

  gio.kicad_pcb      board layout (current iteration)
  gio.kicad_pro      project file
  gio.kicad_sch      schematic (renamed from gio-opamp.kicad_sch)
  gio.kicad_dru      custom design rules
  gio.kicad_mod      custom footprint
  gio-logo.kicad_mod logo footprint for silkscreen

Also added module-logo assets:
  assets/gio.png.gif
  assets/gio.svg

.gitignore extended to exclude KiCad fab/cruft that's regenerated
from the .kicad_pcb on demand:
  *.step             3D model exports (~6 MB each)
  tmp*.rpt           DRC / ERC scratch reports
  _autosave-*        in-flight autosaves
  **/gerber/         Gerber output directory
  **/jlcpcb/         JLC submission directory (project.db, etc.)
  **/production_files/
  *.gbr / *.gbrjob   stray gerber files
  *.drl              drill files
  project.db         KiCad project DB (auto-managed)

The old hardware/gio-opamp/ directory is left on disk untracked --
contains stale duplicates of the renamed files. Safe to rm -rf when
you're sure nothing valuable is in there.

Co-Authored-By: Claude Opus 4.7 (1M context) <noreply@anthropic.com>
Parts:
- removed U4: XIAO-RP2350-DIP, Seeed Studio XIAO Series Library:XIAO-RP2350-DIP, symbol Seeed_Studio_XIAO_Series:XIAO-RP2350-DIP
- added U8: XIAO-RP2350-DIP_pins_only, my_kicad_library:XIAO-RP2350-DIP_pins_only, symbol my_kicad_library:XIAO-RP2350-DIP_pins_only
- C1, C10, C11, C12, C13, C14, C2, C3, C4, C5, C6, C7, C8, C9: footprint Capacitor_SMD:C_0805_2012Metric -> Capacitor_SMD:C_0603_1608Metric
- J3: footprint Connector_PinHeader_1.27mm:PinHeader_1x04_P1.27mm_Vertical -> Connector_PinSocket_2.54mm:PinSocket_1x04_P2.54mm_Vertical
- J4: footprint Connector_PinHeader_2.54mm:PinHeader_1x04_P2.54mm_Vertical -> Connector_IDC:IDC-Header_2x05_P2.54mm_Vertical
- R1, R10, R11, R12, R13, R14, R15, R16, R17, R18, R2, R21, R22, R3, R4, R5, R6, R9: footprint Resistor_SMD:R_0805_2012Metric -> Resistor_SMD:R_0603_1608Metric
- R19, R20, R7, R8: value 14.7k -> 15k; footprint Resistor_SMD:R_0805_2012Metric -> Resistor_SMD:R_0603_1608Metric
- U6: footprint Package_TO_SOT_SMD:TO-252-3_TabPin2 -> Package_TO_SOT_SMD:SOT-223
Connections:
- net +12V: now also J4.10 (Pin_10), J4.9 (Pin_9); no longer J4.1 (Pin_1), J4.2 (Pin_2)
- net +3.3V: now also U8.12 (3V3)
- net +5V: now also U8.14 (VBUS)
- net -12V: now also J4.1 (Pin_1), J4.2 (Pin_2); no longer J4.10 (Pin_10), J4.9 (Pin_9)
- net CS_ADC: now also U8.7 (GPIO0_D6_TXO)
- net CS_DAC: now also U8.4 (GPIO5_D3_SPI0_CS)
- net ENCODER_A: now also U8.2 (GPIO27_A1_D1)
- net ENCODER_B: now also U8.3 (GPIO28_A2_D2)
- net ENCODER_CLICK: now also U8.8 (GPIO1_D7_RX0)
- net GND: now also U8.13 (GND)
- net I2C_SCL: now also U8.6 (GPIO7_D5_SCL1)
- net I2C_SDA: now also U8.5 (GPIO6_D4_SDA1)
- net SPI_MISO: now also U8.10 (GPIO4_D9_SPI0_MISO)
- net SPI_MOSI: now also U8.11 (GPIO3_D10_SPI0_MOSI)
- net SPI_SCK: now also U8.9 (GPIO2_D8_SPI0_SCK)
- no-connect marks 20 -> 10
