File: hardware/gio/gio.kicad_sch (KiCad schematic)
At the start: 55 parts, among them J1 PJ3001F, J2 PJ3001F, J3 oled, J4 eurorack power, J5 PJ3001F, J6 PJ3001F, SW1 encoder, U1 TL072, U2 MCP3208, U3 DAC8552, U5 TL072, U6 AMS1117CD-5.0, U7 REF3040, U8 XIAO-RP2350-DIP_pins_only

Commit message: Hardware Rev 1.1: PCB routing finalized + schematic wire cleanup
Rev 1.1 captures the PCB layout state the user is ready to manufacture
the next batch from. Builds on the Rev 1 bring-up findings (board
electrically validated end-to-end; OLED footprint bug + ADC input
protection captured as Rev 2 to-do items in docs/bench-log.md).

Co-Authored-By: Claude Opus 4.7 (1M context) <noreply@anthropic.com>
Connections:
- net +3.3V: now also J3.2 (Pin_2); no longer J3.3 (Pin_3)
- net GND: now also J3.1 (Pin_1); no longer J3.4 (Pin_4)
- net I2C_SCL: now also J3.3 (Pin_3); no longer J3.2 (Pin_2)
- net I2C_SDA: now also J3.4 (Pin_4); no longer J3.1 (Pin_1)
Other:
- moved on the sheet: J3
Changed lines of the file:
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@@
 	(wire
 		(pts
+			(xy 240.03 135.89) (xy 250.19 135.89)
+		)
+		(stroke
+			(width 0)
+			(type default)
+		)
+	)
+	(wire
+		(pts
 			(xy 232.41 52.07) (xy 232.41 55.88)
 		)
@@
 	(wire
 		(pts
+			(xy 240.03 143.51) (xy 254 143.51)
+		)
+		(stroke
+			(width 0)
+			(type default)
+		)
+	)
+	(wire
+		(pts
 			(xy 95.25 27.94) (xy 99.06 27.94)
 		)
@@
 	(wire
 		(pts
-			(xy 254 146.05) (xy 254 148.59)
+			(xy 254 143.51) (xy 254 148.59)
 		)
 		(stroke
@@
 	(wire
 		(pts
-			(xy 240.03 140.97) (xy 250.19 140.97)
-		)
-		(stroke
-			(width 0)
-			(type default)
-		)
-	)
-	(wire
-		(pts
 			(xy 34.29 29.21) (xy 39.37 29.21)
 		)
@@
 	(wire
 		(pts
-			(xy 254 143.51) (xy 254 132.08)
+			(xy 254 132.08) (xy 254 140.97)
 		)
 		(stroke
@@
 	(wire
 		(pts
-			(xy 240.03 146.05) (xy 254 146.05)
-		)
-		(stroke
-			(width 0)
-			(type default)
-		)
-	)
-	(wire
-		(pts
 			(xy 54.61 111.76) (xy 54.61 115.57)
 		)
@@
 	(wire
 		(pts
-			(xy 240.03 138.43) (xy 250.19 138.43)
-		)
-		(stroke
-			(width 0)
-			(type default)
-		)
-	)
-	(wire
-		(pts
 			(xy 96.52 82.55) (xy 99.06 82.55)
 		)
@@
 	(wire
 		(pts
-			(xy 240.03 143.51) (xy 254 143.51)
+			(xy 240.03 138.43) (xy 250.19 138.43)
 		)
 		(stroke
@@
 	(wire
 		(pts
+			(xy 240.03 140.97) (xy 254 140.97)
+		)
+		(stroke
+			(width 0)
+			(type default)
+		)
+	)
+	(wire
+		(pts
 			(xy 165.1 151.13) (xy 177.8 151.13)
 		)
@@
 		)
 	)
-	(label "I2C_SCL"
-		(at 250.19 140.97 180)
-		(effects
-			(font
-				(size 1.27 1.27)
-			)
-			(justify right bottom)
-		)
-	)
 	(label "SPI_MISO"
 		(at 177.8 146.05 180)
@@
 	)
 	(label "I2C_SDA"
-		(at 250.19 138.43 180)
+		(at 250.19 135.89 180)
 		(effects
 			(font
@@
 		)
 	)
+	(label "I2C_SCL"
+		(at 250.19 138.43 180)
+		(effects
+			(font
+				(size 1.27 1.27)
+			)
+			(justify right bottom)
+		)
+	)
 	(label "SPI_MOSI"
 		(at 184.15 137.16 0)
@@
 		(lib_id "Connector:Conn_01x04_Pin")
 		(at 234.95 140.97 0)
+		(mirror x)
 		(unit 1)
 		(body_style 1)
@@
 		(in_pos_files yes)
 		(dnp no)
-		(fields_autoplaced yes)
 		(property "Reference" "J3"
-			(at 235.585 133.35 0)
+			(at 235.585 148.59 0)
 			(show_name no)
 			(do_not_autoplace no)
@@
 		)
 		(property "Value" "oled"
-			(at 235.585 135.89 0)
+			(at 235.585 146.05 0)
 			(show_name no)
 			(do_not_autoplace no)
